Commit message: Update titatit

File: resources/robots/titatit/urdf/wheeled_titatit_rl.urdf (robot description, URDF)
Before this commit: robot wheeled_titatit_description, 19 links, 18 joints
Links:
- link trunk: geometry collision box size=1.021961 0.312461 0.209650; visual mesh filename=../dae/base.dae
